Commit message: Update and add packages for engineer 2026.

File: engineer2_arm_config/config/gazebo_engineer2.urdf (robot description, URDF)
Before this commit: robot engineer2, 68 links, 67 joints
Links:
- removed link fake_link4
- removed link left_back_roller_0
- removed link left_back_roller_1
- removed link left_back_roller_10
- removed link left_back_roller_11
- removed link left_back_roller_12
- removed link left_back_roller_13
- removed link left_back_roller_2
- removed link left_back_roller_3
- removed link left_back_roller_4
- removed link left_back_roller_5
- removed link left_back_roller_6
- removed link left_back_roller_7
- removed link left_back_roller_8
- removed link left_back_roller_9
- removed link left_front_roller_0
- removed link left_front_roller_1
- removed link left_front_roller_10
- removed link left_front_roller_11
- removed link left_front_roller_12
- removed link left_front_roller_13
- removed link left_front_roller_2
- removed link left_front_roller_3
- removed link left_front_roller_4
- removed link left_front_roller_5
- removed link left_front_roller_6
- removed link left_front_roller_7
- removed link left_front_roller_8
- removed link left_front_roller_9
- removed link right_back_roller_0
- removed link right_back_roller_1
- removed link right_back_roller_10
- removed link right_back_roller_11
- removed link right_back_roller_12
- removed link right_back_roller_13
- removed link right_back_roller_2
- removed link right_back_roller_3
- removed link right_back_roller_4
- removed link right_back_roller_5
- removed link right_back_roller_6
- removed link right_back_roller_7
- removed link right_back_roller_8
- removed link right_back_roller_9
- removed link right_front_roller_0
- removed link right_front_roller_1
- removed link right_front_roller_10
- removed link right_front_roller_11
- removed link right_front_roller_12
- removed link right_front_roller_13
- removed link right_front_roller_2
- removed link right_front_roller_3
- removed link right_front_roller_4
- removed link right_front_roller_5
- removed link right_front_roller_6
- removed link right_front_roller_7
- removed link right_front_roller_8
- removed link right_front_roller_9
- added link exchange_orientation
- added link gripper_link, mass 0.033278; collision mesh filename=package://rm_description/meshes/engineer2/gripper_link.stl; visual mesh filename=package://rm_description/meshes/engineer2/gripper_link.stl
- added link left_lifter, mass 2.255732; collision mesh filename=package://rm_description/meshes/engineer2/left_lifter.stl; visual mesh filename=package://rm_description/meshes/engineer2/left_lifter.stl
- added link left_lifter_wheel, mass 0.120935; collision mesh filename=package://rm_description/meshes/engineer2/left_lifter_wheel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; visual mesh filename=package://rm_description/meshes/engineer2/left_lifter_wheel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
- added link link7, mass 1.6955; collision mesh filename=package://rm_description/meshes/engineer2/link7.stl; visual mesh filename=package://rm_description/meshes/engineer2/link7.stl
- added link right_lifter, mass 2.255732; collision mesh filename=package://rm_description/meshes/engineer2/right_lifter.stl; visual mesh filename=package://rm_description/meshes/engineer2/right_lifter.stl
- added link right_lifter_wheel, mass 0.120935; collision mesh filename=package://rm_description/meshes/engineer2/right_lifter_whee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; visual mesh filename=package://rm_description/meshes/engineer2/right_lifter_whee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
- added link tools_link
- added link yaw
- link base_link: mass 15.736541 -> 34.432921
- link left_back_wheel: geometry collision mesh filename=package://rm_description/meshes/common/left_threaded_14roll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; visual mesh filename=package://rm_description/meshes/common/left_threaded_14roll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
- link left_front_wheel: geometry collision mesh filename=package://rm_description/meshes/common/right_threaded_14rol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; visual mesh filename=package://rm_description/meshes/common/right_threaded_14rol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
- link link1: mass 2.49351 -> 2.95894
- link link2: mass 0.601539 -> 3.65444
- link link3: mass 1.031279 -> 2.313792
- link link4: mass 0.874408 -> 1.745846
- link link5: mass 0.093643 -> 1.488874
- link link6: mass 0.23135 -> 1.22143
- link right_back_wheel: geometry collision mesh filename=package://rm_description/meshes/common/right_threaded_14rol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; visual mesh filename=package://rm_description/meshes/common/right_threaded_14rol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
- link right_front_wheel: geometry collision mesh filename=package://rm_description/meshes/common/left_threaded_14roll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; visual mesh filename=package://rm_description/meshes/common/left_threaded_14roll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
Joints:
- removed joint left_back_roller_0_joint
- removed joint left_back_roller_10_joint
- removed joint left_back_roller_11_joint
- removed joint left_back_roller_12_joint
- removed joint left_back_roller_13_joint
- removed joint left_back_roller_1_joint
- removed joint left_back_roller_2_joint
- removed joint left_back_roller_3_joint
- removed joint left_back_roller_4_joint
- removed joint left_back_roller_5_joint
- removed joint left_back_roller_6_joint
- removed joint left_back_roller_7_joint
- removed joint left_back_roller_8_joint
- removed joint left_back_roller_9_joint
- removed joint left_front_roller_0_joint
- removed joint left_front_roller_10_joint
- removed joint left_front_roller_11_joint
- removed joint left_front_roller_12_joint
- removed joint left_front_roller_13_joint
- removed joint left_front_roller_1_joint
- removed joint left_front_roller_2_joint
- removed joint left_front_roller_3_joint
- removed joint left_front_roller_4_joint
- removed joint left_front_roller_5_joint
- removed joint left_front_roller_6_joint
- removed joint left_front_roller_7_joint
- removed joint left_front_roller_8_joint
- removed joint left_front_roller_9_joint
- removed joint middle_pitch
- removed joint right_back_roller_0_joint
- removed joint right_back_roller_10_joint
- removed joint right_back_roller_11_joint
- removed joint right_back_roller_12_joint
- removed joint right_back_roller_13_joint
- removed joint right_back_roller_1_joint
- removed joint right_back_roller_2_joint
- removed joint right_back_roller_3_joint
- removed joint right_back_roller_4_joint
- removed joint right_back_roller_5_joint
- removed joint right_back_roller_6_joint
- removed joint right_back_roller_7_joint
- removed joint right_back_roller_8_joint
- removed joint right_back_roller_9_joint
- removed joint right_front_roller_0_joint
- removed joint right_front_roller_10_joint
- removed joint right_front_roller_11_joint
- removed joint right_front_roller_12_joint
- removed joint right_front_roller_13_joint
- removed joint right_front_roller_1_joint
- removed joint right_front_roller_2_joint
- removed joint right_front_roller_3_joint
- removed joint right_front_roller_4_joint
- removed joint right_front_roller_5_joint
- removed joint right_front_roller_6_joint
- removed joint right_front_roller_7_joint
- removed joint right_front_roller_8_joint
- removed joint right_front_roller_9_joint
- added joint exchange_orientation_joint: type fixed, parent base_link, child exchange_orientation, origin xyz=0.0 0.0 0.0 rpy=0.0 0.0 -1.57
- added joint gripper_joint: type revolute, parent link7, child gripper_link, origin xyz=0. -0.05625 0. rpy=0 0 0, axis 0 1 0, limit lower=0.27 upper=1.15 effort=7 velocity=20.94
- added joint joint7: type revolute, parent link6, child link7, origin xyz=0. 0.007 0. rpy=0 0 0, axis 0 1 0, limit lower=-2.6 upper=2.73 effort=7 velocity=20.94
- added joint left_lifter_joint: type prismatic, parent base_link, child left_lifter, origin xyz=-0.282 0.275 0.460 rpy=0 0 0, axis 0 0 1, limit lower=0 upper=0.22 effort=259.2 velocity=1.0
- added joint left_lifter_wheel_joint: type continuous, parent left_lifter, child left_lifter_wheel, origin xyz=0.007 -0.575 -0.2385 rpy=0 0 0, axis 1 0 0, limit effort=2 velocity=25
- added joint right_lifter_joint: type prismatic, parent base_link, child right_lifter, origin xyz=0.282 0.275 0.460 rpy=0 0 0, axis 0 0 1, limit lower=0 upper=0.22 effort=259.2 velocity=1.0
- added joint right_lifter_wheel_joint: type continuous, parent right_lifter, child right_lifter_wheel, origin xyz=0.007 -0.575 -0.2385 rpy=0 0 0, axis 1 0 0, limit effort=2 velocity=25
- added joint tools_joint: type fixed, parent gripper_link, child tools_link, origin xyz=0.1 0. 0. rpy=0 0 0
- added joint yaw_joint: type fixed, parent base_link, child yaw, origin xyz=0. 0. 1. rpy=0 0 0, axis 0 0 1
- joint joint1: limit lower=0 upper=0.3 effort=1000 velocity=2.25 -> lower=0 upper=0.552 effort=300 velocity=1.929; origin xyz=0. 0. 0.260 rpy=0 0 0 -> xyz=-0.008 0.189 0.25475 rpy=0 0 0
- joint joint2: limit lower=-1.2 upper=1.2 effort=40 velocity=10.46 -> lower=-3.41 upper=1.66 effort=25 velocity=3.76; origin xyz=0.082 -0.2 0. rpy=0 0 0 -> xyz=-0.040998 -0.390478 0.0083 rpy=0 0 0
- joint joint3: axis 0 0 1 -> 1 0 0; limit lower=-1.2 upper=1.2 effort=25 velocity=3.76 -> lower=-1.07 upper=1.32 effort=40 velocity=10.46; origin xyz=0.275 0. 0. rpy=0 0 0 -> xyz=-0.0379 0. 0.08495 rpy=0 0 0
- joint joint4: limit lower=-3.14 upper=3.14 effort=7 velocity=20.94 -> lower=-3.43 upper=1.01 effort=25 velocity=3.76; origin xyz=0.153 0. 0.086605 rpy=0 0 0 -> xyz=0.004999 0. 0.185 rpy=0 0 0
- joint joint5: limit lower=-1.57 upper=1.57 effort=14 velocity=10 -> lower=-2.13 upper=2.05 effort=7 velocity=20.94; origin xyz=0.1055 0.0 0. rpy=0 0 0 -> xyz=0.032901 -0.128 0. rpy=0 0 0
- joint joint6: limit lower=-6 upper=6 effort=14 velocity=10 -> lower=-1.9 upper=1.83 effort=7 velocity=20.94; origin xyz=0.026183 0 0 rpy=0 0 0 -> xyz=0. -0.147 0. rpy=0 0 0
